File: ESP32_Core.kicad_sch (KiCad schematic)
At the start: 30 parts, among them J2 USB_C_Receptacle_USB2.0_16P, J28 Conn_01x03, J29 Conn_01x03, J30 Conn_01x03, J31 Conn_01x03, J32 Conn_01x03, J33 Conn_01x03, J34 Conn_01x03, J35 Conn_01x03, J36 Conn_01x03, J37 Conn_01x03, J38 Conn_01x03, J39 Conn_01x03, SW2 SW_Push, SW3 SW_Push, U1 ESP32-WROOM-32, U2 CP2102N-Axx-xQFN20

Commit message: Add files via upload
Checkpoint: schematic through USB programming power section
Connections:
- net DS18B20_DQ: now reaches U1.29 (IO5)
- net FLAME_AO_ADC: now reaches U1.4 (SENSOR_VP)
- net INA226_ALERT: now reaches U1.5 (SENSOR_VN)
- no-connect marks 21 -> 18
Changed lines of the file:
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@@
-	)
-	(no_connect
-		(at 46.99 44.45)
 	)
 	(no_connect
@@
 	)
 	(no_connect
-		(at 46.99 46.99)
-	)
-	(no_connect
 		(at 46.99 74.93)
 	)
@@
 	)
 	(no_connect
-		(at 77.47 52.07)
-	)
-	(no_connect
 		(at 124.46 64.77)
 	)
@@
 		(pts
 			(xy 199.39 105.41) (xy 199.39 107.95)
+		)
+		(stroke
+			(width 0)
+			(type default)
+		)
+	)
+	(wire
+		(pts
+			(xy 35.56 44.45) (xy 46.99 44.45)
 		)
 		(stroke
@@
 			)
 			(justify right bottom)
+		)
+	)
+	(global_label "DS18B20_DQ"
+		(shape input)
+		(at 77.47 52.07 0)
+		(fields_autoplaced yes)
+		(effects
+			(font
+				(size 1.27 1.27)
+			)
+			(justify left)
+		)
+		(property "Intersheetrefs" "${INTERSHEET_REFS}"
+			(at 92.6108 52.07 0)
+			(hide yes)
+			(show_name no)
+			(do_not_autoplace no)
+			(effects
+				(font
+					(size 1.27 1.27)
+				)
+				(justify left)
+			)
+		)
+	)
+	(global_label "INA226_ALERT"
+		(shape input)
+		(at 46.99 46.99 180)
+		(fields_autoplaced yes)
+		(effects
+			(font
+				(size 1.27 1.27)
+			)
+			(justify right)
+		)
+		(property "Intersheetrefs" "${INTERSHEET_REFS}"
+			(at 30.8815 46.99 0)
+			(hide yes)
+			(show_name no)
+			(do_not_autoplace no)
+			(effects
+				(font
+					(size 1.27 1.27)
+				)
+				(justify right)
+			)
 		)
 	)
@@
 			)
 		)
+	)
+	(global_label "FLAME_AO_ADC"
+		(shape input)
+		(at 35.56 44.45 180)
+		(fields_autoplaced yes)
+		(effects
+			(font
+				(size 1.27 1.27)
+			)
+			(justify right)
+		)
+		(property "Intersheetrefs" "${INTERSHEET_REFS}"
+			(at 18.7862 44.45 0)
+			(hide yes)
+			(show_name no)
+			(do_not_autoplace no)
+			(effects
+				(font
+					(size 1.27 1.27)
+				)
+				(justify right)
+			)
+		)
