File: Environment_Sensors.kicad_sch (KiCad schematic)
At the start: 14 parts, among them J3 Conn_01x04_Pin, U5 VL53L0CXV0DH1, U7 MQ-2

Commit message: Add files via upload
Checkpoint: schematic through USB programming power section
Parts:
- added C15: 100nF, symbol Device:C_Small
- added R16: 4.7k, symbol Device:R
- added R17, R18: 2.2k, symbol Device:R
- added U6: DS18B20, Package_TO_SOT_THT:TO-92_Inline, symbol Sensor_Temperature:DS18B20
- added U8: TCA9548APWR, Package_SO:TSSOP-24_4.4x7.8mm_P0.65mm, symbol Interface_Expansion:TCA9548APWR
Connections:
- net +3V3: now also C15.1, R16.2, R17.1, R18.1, U6.3 (V_{DD}), U8.24 (VCC), U8.3 (~{RESET})
- net BNO055_SCL: now also U8.22 (SCL); no longer U5.10 (SCL)
- net BNO055_SDA: now also U8.23 (SDA); no longer U5.9 (SDA)
- net GND: now also C15.2, U6.1 (GND), U8.1 (A0), U8.12 (GND), U8.2 (A1), U8.21 (A2)
- new net DS18B20_DQ: R16.1, U6.2 (DQ)
- new net VL53_SCL: R18.2, U5.10 (SCL), U8.5 (SC0)
- new net VL53_SDA: R17.2, U5.9 (SDA), U8.4 (SD0)
- no-connect marks 0 -> 14
