File: Power_Monitor.kicad_sch (KiCad schematic)
At the start: 0 parts

Commit message: Add files via upload
Checkpoint: schematic through USB programming power section
Parts:
- added C16: 100nF, symbol Device:C_Small_US
- added R19: 1mΩ 5W, symbol Device:R_Shunt
- added R20: 10k, symbol Device:R
- added U9: INA226, Package_SO:TSSOP-10_3x3mm_P0.5mm, symbol Sensor_Energy:INA226
Connections:
- new net +3V3: C16.1, R20.2, U9.6 (VS)
- new net +5V: R19.1, U9.10 (Vin+)
- new net BNO055_SCL: U9.5 (SCL)
- new net BNO055_SDA: U9.4 (SDA)
- new net GND: C16.2, U9.1 (A1), U9.2 (A0), U9.7 (GND)
- new net INA226_ALERT: R20.1, U9.3 (~{Alert})
- new net SERVO_5V: R19.4, U9.8 (Vbus), U9.9 (Vin-)
