File: USB_Programming.kicad_sch (KiCad schematic)
At the start: 0 parts

Commit message: Add files via upload
Checkpoint: schematic through USB programming power section
Parts:
- added C17: 1uF, symbol Device:C_Small
- added U10: CP2102N-Axx-xQFN24, Package_DFN_QFN:QFN-24-1EP_4x4mm_P0.5mm_EP2.6x2.6mm, symbol Interface_USB:CP2102N-Axx-xQFN24
Connections:
- new net: C17.1, U10.6 (VDD)
- new net +3V3: U10.5 (VIO)
- new net +5V: U10.7 (VREGIN), U10.8 (VBUS)
- new net GND: C17.2, U10.2 (GND), U10.25 (GND)
